File: Eagle_Project/Decoder_SMD/CAB_decoder_SMD_rev2.kicad_sch (KiCad schematic)
At the start: 43 parts, among them IC1 TLE5206-2G, Q1 BSS138, Q2 BSS138, Q3 BSS138, Q4 BSS138, Q5 BSS138, Q6 BSS138

Commit message: esp32_decoder kicad setup
Parts:
- removed ARDUINO_NANO1: ARDUINO_NANO, toytrains_decoder_smd:ARDUINO_NANO, symbol toytrains_decoder_smd-eagle-import:ArduinoNanoV30_ARDUINO_NANO
- removed AUX-5V-1, AUX-5V-2: 5V_OUT, toytrains_decoder_smd:MOLEX-1X2_LOCK, symbol toytrains_decoder_smd-eagle-import:SparkFun-Connectors_513_CONN_02POLAR_LOCK
- removed B2-RECTIFIER0: 2w10, toytrains_decoder_smd:1KAB, symbol toytrains_decoder_smd-eagle-import:rectifier_336_1KAB
- removed C1: 470uF 35V, toytrains_decoder_smd:153CLV-1014, symbol toytrains_decoder_smd-eagle-import:rcl_334_CPOL-EU153CLV-1014
- removed C2: 100uF 10V, toytrains_decoder_smd:153CLV-0605, symbol toytrains_decoder_smd-eagle-import:rcl_334_CPOL-EU153CLV-0605
- removed C4, C5, C6, C9: 0.1uF, toytrains_decoder_smd:C1206, symbol toytrains_decoder_smd-eagle-import:rcl_334_C-EUC1206
- removed C7, C8: 22uF 16V, toytrains_decoder_smd:153CLV-0405, symbol toytrains_decoder_smd-eagle-import:rcl_334_CPOL-EU153CLV-0405
- removed D1, D2: MINIMELF, toytrains_decoder_smd:MINIMELF, symbol toytrains_decoder_smd-eagle-import:diode_210_DIODE-MINIMELF
- removed D1-1N5817: S1, toytrains_decoder_smd:DO214AC, symbol toytrains_decoder_smd-eagle-import:s1x_10_S1
- removed DCC-IN0, F1, F2, F3, F4, F5, F6, MOTOR_OUT1: CONN_02POLAR_LOCK, toytrains_decoder_smd:MOLEX-1X2_LOCK, symbol toytrains_decoder_smd-eagle-import:SparkFun-Connectors_513_CONN_02POLAR_LOCK
- removed IC1: TLE5206-2G, toytrains_decoder_smd:P-TO263-7-1, symbol toytrains_decoder_smd-eagle-import:HBridge_TLE5206-2G
- removed OK1: HCPL0601, toytrains_decoder_smd:SOIC08, symbol toytrains_decoder_smd-eagle-import:optocoupler_320_HCPL0601
- removed POWER-LED0: LEDCHIPLED_1206, toytrains_decoder_smd:CHIPLED_1206, symbol toytrains_decoder_smd-eagle-import:led_259_LEDCHIPLED_1206
- removed Q1, Q2, Q3, Q4, Q5, Q6: BSS138, toytrains_decoder_smd:SOT23, symbol toytrains_decoder_smd-eagle-import:bss138_10_BSS138
- removed R1, R2: 430Ω, toytrains_decoder_smd:R2512, symbol toytrains_decoder_smd-eagle-import:rcl_334_R-EU_R2512
- removed R10, R9: 10kΩ, toytrains_decoder_smd:R1206, symbol toytrains_decoder_smd-eagle-import:rcl_334_R-EU_R1206
- removed R11, R7, R8: 2.2kΩ, toytrains_decoder_smd:R1206, symbol toytrains_decoder_smd-eagle-import:rcl_334_R-EU_R1206
- removed R15: 560Ω, toytrains_decoder_smd:R1206, symbol toytrains_decoder_smd-eagle-import:rcl_334_R-EU_R1206
- removed R3: 1kΩ, toytrains_decoder_smd:R1206, symbol toytrains_decoder_smd-eagle-import:rcl_334_R-EU_R1206
- removed U$1: LM2594, toytrains_decoder_smd:SOIC8, symbol toytrains_decoder_smd-eagle-import:LM2594_LM2594
- removed U$2: L-CD54, toytrains_decoder_smd:L_CD54, symbol toytrains_decoder_smd-eagle-import:Inductor_L-CD54
- added ARDUINO_NANO1: ARDUINO_NANO, CAB_decoder_SMD:ARDUINO_NANO, symbol CAB_decoder_SMD-eagle-import:ARDUINO_NANO
- added AUX-5V-1, AUX-5V-2: 5V_OUT, CAB_decoder_SMD:MOLEX-1X2_LOCK, symbol CAB_decoder_SMD-eagle-import:CONN_02POLAR_LOCK
- added B2-RECTIFIER0: 2w10, CAB_decoder_SMD:1KAB, symbol CAB_decoder_SMD-eagle-import:1KAB
- added C1: 470uF 35V, CAB_decoder_SMD:153CLV-1014, symbol CAB_decoder_SMD-eagle-import:CPOL-EU153CLV-1014
- added C2: 100uF 10V, CAB_decoder_SMD:153CLV-0605, symbol CAB_decoder_SMD-eagle-import:CPOL-EU153CLV-0605
- added C4, C5, C6, C9: 0.1uF, CAB_decoder_SMD:C1206, symbol CAB_decoder_SMD-eagle-import:C-EUC1206
- added C7, C8: 22uF 16V, CAB_decoder_SMD:153CLV-0405, symbol CAB_decoder_SMD-eagle-import:CPOL-EU153CLV-0405
- added D1, D2: MINIMELF, CAB_decoder_SMD:MINIMELF, symbol CAB_decoder_SMD-eagle-import:DIODE-MINIMELF
- added D1-1N5817: S1, CAB_decoder_SMD:DO214AC, symbol CAB_decoder_SMD-eagle-import:S1
- added DCC-IN0, F1, F2, F3, F4, F5, F6, MOTOR_OUT1: CONN_02POLAR_LOCK, CAB_decoder_SMD:MOLEX-1X2_LOCK, symbol CAB_decoder_SMD-eagle-import:CONN_02POLAR_LOCK
- added IC1: TLE5206-2G, CAB_decoder_SMD:P-TO263-7-1, symbol CAB_decoder_SMD-eagle-import:TLE5206-2G
- added OK1: HCPL0601, CAB_decoder_SMD:SOIC08, symbol CAB_decoder_SMD-eagle-import:HCPL0601
- added POWER-LED0: LEDCHIPLED_1206, CAB_decoder_SMD:CHIPLED_1206, symbol CAB_decoder_SMD-eagle-import:LEDCHIPLED_1206
- added Q1, Q2, Q3, Q4, Q5, Q6: BSS138, CAB_decoder_SMD:SOT23, symbol CAB_decoder_SMD-eagle-import:BSS138
- added R1, R2: 430Ω, CAB_decoder_SMD:R2512, symbol CAB_decoder_SMD-eagle-import:R-EU_R2512
- added R10, R9: 10kΩ, CAB_decoder_SMD:R1206, symbol CAB_decoder_SMD-eagle-import:R-EU_R1206
- added R11, R7, R8: 2.2kΩ, CAB_decoder_SMD:R1206, symbol CAB_decoder_SMD-eagle-import:R-EU_R1206
- added R15: 560Ω, CAB_decoder_SMD:R1206, symbol CAB_decoder_SMD-eagle-import:R-EU_R1206
- added R3: 1kΩ, CAB_decoder_SMD:R1206, symbol CAB_decoder_SMD-eagle-import:R-EU_R1206
- added U$2: L-CD54, CAB_decoder_SMD:L_CD54, symbol CAB_decoder_SMD-eagle-import:L-CD54
- added U1: LM2596T-5, Package_TO_SOT_THT:TO-220-5_P3.4x3.7mm_StaggerOdd_Lead3.8mm_Vertical, symbol Regulator_Switching:LM2596T-5
Connections:
- net GND: now also ARDUINO_NANO1.19 (GND@1), AUX-5V-1.2, AUX-5V-2.2, B2-RECTIFIER0.-, C1.-, C2.-, C4.1, C5.2, C9.2, D1-1N5817.A, IC1.4 (GND), IC1.8 (GND), OK1.5 (GND), POWER-LED0.C, Q1.2 (S), Q2.2 (S), Q3.2 (S), Q4.2 (S), Q5.2 (S), Q6.2 (S), R8.2
- net VIN: now also ARDUINO_NANO1.15 (VIN)
- new net: ARDUINO_NANO1.5 (A1), C6.1, C7.+, R8.1, R9.2
- new net: C6.2, C7.-
- new net: AUX-5V-1.1, AUX-5V-2.1, C2.+, C5.1, D1.A, F1.1, F2.1, F3.1, F4.1, F5.1, F6.1, OK1.7 (VE), OK1.8 (VCC), R11.1, R15.1, R3.2, U$2.P$2
- new net: F1.2, Q6.3 (D)
- new net: ARDUINO_NANO1.6 (A2), IC1.2 (EF), R11.2
- new net: F2.2, Q5.3 (D)
- new net: ARDUINO_NANO1.26 (D8), Q1.1 (G)
- new net: F6.2, Q1.3 (D)
- new net: IC1.1 (OUT1), MOTOR_OUT1.1
- new net: IC1.7 (OUT2), MOTOR_OUT1.2
- new net: B2-RECTIFIER0.AC2, D2.A, DCC-IN0.1, OK1.3 (C), R9.1
- new net: D2.C, OK1.2 (A), R1.1
- new net: POWER-LED0.A, R15.2
- new net: ARDUINO_NANO1.24 (D6), Q3.1 (G)
- new net: F4.2, Q3.3 (D)
- new net: B2-RECTIFIER0.+, C1.+, C9.1, IC1.6 (VS)
- new net: ARDUINO_NANO1.28 (D10), IC1.3 (IN1)
- new net: ARDUINO_NANO1.27 (D9), IC1.5 (IN2)
- new net: ARDUINO_NANO1.20 (D2), OK1.6 (VO), R3.1
- new net: B2-RECTIFIER0.AC1, DCC-IN0.2, R10.1, R2.2
- new net: F5.2, Q2.3 (D)
- new net: ARDUINO_NANO1.25 (D7), Q2.1 (G)
- new net: ARDUINO_NANO1.22 (D4), Q5.1 (G)
- new net: ARDUINO_NANO1.4 (A0), C4.2, C8.+, R10.2, R7.1
- new net: R1.2, R2.1
- new net: ARDUINO_NANO1.21 (D3), Q6.1 (G)
- new net: ARDUINO_NANO1.12 (5V), D1.C
- new net: ARDUINO_NANO1.23 (D5), Q4.1 (G)
- new net: F3.2, Q4.3 (D)
